Commit message: switched default to obj

File: urdf/arm/openarm_arm.xacro (robot description, xacro)
@@ -2,5 +2,5 @@
 <robot xmlns:xacro="http://www.ros.org/wiki/xacro" name="openarm">
   <xacro:include filename="$(find openarm_description)/urdf/arm/openarm_macro.xacro" />
-  <xacro:macro name="openarm_arm" params="arm_type arm_prefix:='' no_prefix:=false description_pkg:='openarm_description' connected_to:='base' xyz:='0 0 0' rpy:='0 0 0' joint_limits inertials kinematics kinematics_link kinematics_offset:=none mesh_ext:='dae'" >
+  <xacro:macro name="openarm_arm" params="arm_type arm_prefix:='' no_prefix:=false description_pkg:='openarm_description' connected_to:='base' xyz:='0 0 0' rpy:='0 0 0' joint_limits inertials kinematics kinematics_link kinematics_offset:=none mesh_ext:='obj'" >
     <xacro:property name="prefix" value="${'' if no_prefix else 'openarm' + '_' + arm_prefix}" />
     <xacro:if value="${arm_prefix == 'right_'}">

File: urdf/body/openarm_body.xacro (robot description, xacro)
@@ -13,5 +13,5 @@
               kinematics
               kinematics_link
-              mesh_ext:='dae'
+              mesh_ext:='obj'
               ">
     <!-- <xacro:property name="prefix" value="${'' if no_prefix else body_prefix + 'body_'}" /> -->

File: urdf/ee/ee_with_one_link.xacro (robot description, xacro)
@@ -2,5 +2,5 @@
 <robot xmlns:xacro="http://www.ros.org/wiki/xacro" name="ee_with_one_link">
   <!-- safety_distance: Minimum safety distance in [m] by which the collision volumes are expanded and which is enforced during robot motions -->
-  <xacro:macro name="ee_with_one_link" params="connected_to:='' arm_type arm_prefix:='' ee_type ee_inertials rpy_ee:='0 0 0' xyz_ee:='0 0 0' tcp_xyz:='0 0 0' tcp_rpy:='0 0 0' description_pkg:=openarm_description with_sc:=false mesh_ext:='dae'">
+  <xacro:macro name="ee_with_one_link" params="connected_to:='' arm_type arm_prefix:='' ee_type ee_inertials rpy_ee:='0 0 0' xyz_ee:='0 0 0' tcp_xyz:='0 0 0' tcp_rpy:='0 0 0' description_pkg:=openarm_description with_sc:=false mesh_ext:='obj'">
     <xacro:property name="ee_prefix" default="robot_"/>
     <xacro:unless value="${arm_type == ''}">

File: urdf/ee/openarm_hand.xacro (robot description, xacro)
@@ -2,5 +2,5 @@
 <robot xmlns:xacro="http://www.ros.org/wiki/xacro" name="hand">
   <!-- safety_distance: Minimum safety distance in [m] by which the collision volumes are expanded and which is enforced during robot motions -->
-  <xacro:macro name="openarm_hand" params="connected_to:='' arm_type arm_prefix:='' ee_type ee_inertials ee_kinematics_link rpy_ee:='0 0 0' xyz_ee:='0 0 0' tcp_xyz:='0 0 0' tcp_rpy:='0 0 0' description_pkg:=openarm_description mesh_ext:='dae'">
+  <xacro:macro name="openarm_hand" params="connected_to:='' arm_type arm_prefix:='' ee_type ee_inertials ee_kinematics_link rpy_ee:='0 0 0' xyz_ee:='0 0 0' tcp_xyz:='0 0 0' tcp_rpy:='0 0 0' description_pkg:=openarm_description mesh_ext:='obj'">
     <xacro:property name="ee_prefix" default=""/>
     <xacro:unless value="${arm_type == ''}">

File: urdf/robot/openarm_robot.xacro (robot description, xacro)
@@ -36,5 +36,5 @@
             left_arm_prefix:='left_'
             right_arm_prefix:='right_'
-            mesh_ext:='dae'
+            mesh_ext:='obj'
             ">
     <xacro:include filename="$(find openarm_description)/urdf/arm/openarm_macro.xacro" />

File: urdf/robot/v10.urdf.xacro (robot description, xacro)
@@ -22,5 +22,5 @@
   <xacro:arg name="fake_sensor_commands" default="false" />
   <xacro:arg name="bimanual" default="false" />
-  <xacro:arg name="mesh_ext" default="dae" />
+  <xacro:arg name="mesh_ext" default="obj" />
   <xacro:arg name="right_arm_base_xyz" default="0.0 -0.031 0.698" />
   <xacro:arg name="right_arm_base_rpy" default="1.5708 0 0" />
